File: SeCloud.sch (EAGLE design)
At the start: 92 parts, among them Q1 E4SB25.000F20E15(25MHz/20pF/2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, U3 SY6280, U7 MP1482DS, U8 RTL8211CL-GR

Commit message: Added lbr, RTL8188 module, and SATA connector;
Parts:
- removed 5V_SATA_PWR: DW02S, Penko:CON2DW02S
- removed L8: FB0805/600R/2A, rcl:L-USL0805_5MIL_DWS
- removed SATA: SATA-PWA-07, OLIMEX_CONNECTORS:SATA-PWA-07
- removed USB_HOST: USB_TWO_LEVEL, OLIMEX_CONNECTORS:USB_TWO_LEVEL
- added U$1: RTL8188CUS-MOD, SeCloud:RTL8188CUS-MOD
- added U$2: SATA-CON, SeCloud:SATA-CON
- added X1: (no value), con-berg:PN87520
- added X2: BU-SMA-H, con-coax:BU-SMA-H
Connections:
- removed net N$193: L8.2, USB_HOST.GND1, USB_HOST.GND2, USB_HOST.GND3, USB_HOST.GND4
- new net ANT: U$1.ANT, X2.1
- net +5V: now also U$2.5V; no longer 5V_SATA_PWR.1
- net GND: now also U$1.GND, U$1.RF_GND, U$2.GND, X1.4, X2.2; no longer 5V_SATA_PWR.2, L8.1, SATA.GND, SATA.GND@1, SATA.GND@2, USB_HOST.2.4
- net N$106: now also U$2.A+; no longer SATA.A+
- net N$112: now also U$2.A-; no longer SATA.A-
- net N$113: now also U$2.B-; no longer SATA.B-
- net N$114: now also U$2.B+; no longer SATA.B+
- net N$194: now also X1.1; no longer USB_HOST.2.1
- net UDM1: now also U$1.USB-
- net UDM2: now also X1.2; no longer USB_HOST.2.2
- net UDP1: now also U$1.USB+
- net UDP2: now also X1.3; no longer USB_HOST.2.3
- net VCC: now also U$1.3.3V
Other:
- note added: "Fix DVDD33"
- note removed: "+"
- note removed: "-"
- moved on the sheet: C19, C20
